File: bitaxeUltra.kicad_pcb (KiCad board)
At the start: 4 copper layers, 56.5 x 99.8 mm, 137 parts, among them J1 54-00164, J2 Conn_01x02, J3 Conn_01x05, J4 Conn_01x04, J5 TC2030-IDC, J7 Conn_01x02, J8 USB_C_Receptacle_USB2.0, J9 Conn_01x04, Q1 CSD17311Q5, Q2 CSD17311Q5, Q4 2N7002K, SW1 GT-TC029B-H025-L1N, SW2 GT-TC029B-H025-L1N, U1 25MHz, U10 DS4432U+, U11 RT9080-33GJ5, U12 ESP32-S3-WROOM-1, U14 BM1366_mode1, U2 TXB0104RGYR, U5 MCP1824T-1802E, U6 MCP1824T-0802E, U7 EMC2101, U8 INA260, U9 TPS40305, Y1 32.768kHz

Commit message: add fill
Routing:
- added copper zone on B.Cu, net (none)
- added copper zone on F.Cu, net (none)
- added copper zone on In2.Cu, net (none)
Changed lines of the file:
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@@
+    )
+  )
+  (zone (net 0) (net_name "") (layer "F.Cu") (hatch edge 0.5)
+    (priority 4)
+    (connect_pads (clearance 0))
+    (min_thickness 0.25) (filled_areas_thickness no)
+    (fill yes (thermal_gap 0.5) (thermal_bridge_width 0.5) (island_removal_mode 1) (island_area_min 10))
+    (polygon
+      (pts
+        (xy 75.311 46.863)
+        (xy 75.311 148.463)
+        (xy 135.255 148.717)
+        (xy 135.255 46.609)
+      )
     )
   )
@@
     )
   )
+  (zone (net 0) (net_name "") (layer "In2.Cu") (hatch edge 0.5)
+    (priority 5)
+    (connect_pads (clearance 0))
+    (min_thickness 0.25) (filled_areas_thickness no)
+    (fill yes (thermal_gap 0.5) (thermal_bridge_width 0.5) (island_removal_mode 1) (island_area_min 10))
+    (polygon
+      (pts
+        (xy 76.708 46.99)
+        (xy 136.144 46.99)
+        (xy 134.62 148.717)
+        (xy 75.565 147.447)
+      )
+    )
+  )
   (zone (net 8) (net_name "/3V3") (layer "In2.Cu") (hatch edge 0.508)
     (connect_pads (clearance 0.254))
@@
       )
     )
+  )
+  (zone (net 0) (net_name "") (layer "B.Cu") (hatch edge 0.5)
+    (priority 6)
+    (connect_pads (clearance 0))
+    (min_thickness 0.25) (filled_areas_thickness no)
+    (fill yes (thermal_gap 0.5) (thermal_bridge_width 0.5) (island_removal_mode 1) (island_area_min 10))
+    (polygon
+      (pts
+        (xy 75.819 44.323)
+        (xy 134.493 44.45)
+        (xy 134.874 149.225)
+        (xy 75.946 147.828)
+      )
+    )
