File: esp32.kicad_sch (KiCad schematic)
At the start: 26 parts, among them J5 TC2030-IDC, J8 USB_C_Receptacle_USB2.0, J9 Conn_01x04, SW1 GT-TC029B-H025-L1N, SW2 GT-TC029B-H025-L1N, U11 RT9080-33GJ5, U12 ESP32-S3-WROOM-1, Y1 32.768kHz

Commit message: Finish LED layout. Can pass to factory for prototype test
Parts:
- J5: footprint bitaxe:Tag-Connect_TC2030-IDC-NL_2x03_P1.27mm_Vertical -> Connector:Tag-Connect_TC2030-IDC-NL_2x03_P1.27mm_Vertical
- U11: footprint bitaxe:RT9080-33GJ5 -> TSOT-23-5_RIT
- U12: footprint bitaxe:ESP32-S3-WROOM-1 -> Espressif:ESP32-S3-WROOM-1
Changed lines of the file:
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@@
       (effects (font (size 1.27 1.27)) hide)
     )
-    (property "Datasheet" "" (at 35.56 86.995 0)
+    (property "Datasheet" "~" (at 35.56 86.995 0)
       (effects (font (size 1.27 1.27)) hide)
     )
@@
       (effects (font (size 1.27 1.27)) hide)
     )
-    (property "Datasheet" "" (at 132.715 62.23 0)
+    (property "Datasheet" "~" (at 132.715 62.23 0)
       (effects (font (size 1.27 1.27)) hide)
     )
@@
       (effects (font (size 1.27 1.27)))
     )
-    (property "Footprint" "bitaxe:RT9080-33GJ5" (at 100.965 12.7 0)
+    (property "Footprint" "TSOT-23-5_RIT" (at 100.965 12.7 0)
       (effects (font (size 1.524 1.524)) hide)
     )
@@
       (effects (font (size 1.27 1.27)))
     )
-    (property "Footprint" "bitaxe:Tag-Connect_TC2030-IDC-NL_2x03_P1.27mm_Vertical" (at 64.77 168.275 0)
+    (property "Footprint" "Connector:Tag-Connect_TC2030-IDC-NL_2x03_P1.27mm_Vertical" (at 64.77 168.275 0)
       (effects (font (size 1.27 1.27)) hide)
     )
@@
       (effects (font (size 1.27 1.27)) hide)
     )
-    (property "Datasheet" "" (at 69.215 35.56 0)
+    (property "Datasheet" "~" (at 69.215 35.56 0)
       (effects (font (size 1.27 1.27)) hide)
     )
@@
       (effects (font (size 1.27 1.27)) hide)
     )
-    (property "Datasheet" "" (at 121.92 62.23 0)
+    (property "Datasheet" "~" (at 121.92 62.23 0)
       (effects (font (size 1.27 1.27)) hide)
     )
@@
       (effects (font (size 1.27 1.27)) hide)
     )
-    (property "Datasheet" "https://www.sii.co.jp/en/quartz/files/2013/03/SC-32S_Leaflet_e20151217.pdf" (at 137.16 29.845 0)
+    (property "Datasheet" "~" (at 137.16 29.845 0)
       (effects (font (size 1.27 1.27)) hide)
     )
@@
       (effects (font (size 1.27 1.27)) hide)
     )
-    (property "Datasheet" "https://gct.co/connector/usb4105" (at 234.315 69.215 0)
+    (property "Datasheet" "https://www.usb.org/sites/default/files/documents/usb_type-c.zip" (at 234.315 69.215 0)
       (effects (font (size 1.27 1.27)) hide)
     )
@@
       (effects (font (size 1.27 1.27)) hide)
     )
-    (property "Datasheet" "" (at 31.115 35.56 0)
+    (property "Datasheet" "~" (at 31.115 35.56 0)
       (effects (font (size 1.27 1.27)) hide)
     )
@@
       (effects (font (size 1.27 1.27)))
     )
-    (property "Footprint" "bitaxe:ESP32-S3-WROOM-1" (at 133.35 140.97 0)
-      (effects (font (size 1.27 1.27)) hide)
-    )
+    (property "Footprint" "Espressif:ESP32-S3-WROOM-1" (at 133.35 140.97 0)
+      (effects (font (size 1.27 1.27)) hide)
+    )
