File: power.kicad_sch (KiCad schematic)
At the start: 29 parts, among them J7 Conn_01x02, Q1 CSD17311Q5, Q2 CSD17311Q5, Q4 2N7002K, U10 DS4432U+, U8 INA260, U9 TPS40305

Commit message: Finish LED layout. Can pass to factory for prototype test
Parts:
- Q1, Q2: footprint bitaxe:CSD17311Q5 -> TPS40305_supply:CSD17311Q5
- Q4: footprint Package_TO_SOT_SMD:SOT-323_SC-70 -> Package_TO_SOT_SMD:SOT-23
- U9: footprint bitaxe:TPS40305 -> TPS40305_supply:TPS40305
Changed lines of the file:
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@@
       (effects (font (size 1.27 1.27)) hide)
     )
-    (property "Datasheet" "" (at 157.48 62.23 0)
+    (property "Datasheet" "~" (at 157.48 62.23 0)
       (effects (font (size 1.27 1.27)) hide)
     )
@@
       (effects (font (size 1.27 1.27)) hide)
     )
-    (property "Datasheet" "https://media.digikey.com/pdf/Data%20Sheets/Panasonic%20Capacitors%20PDFs/TPE_Series_POSCAP_Rev02_Oct_2017.pdf" (at 230.505 52.705 0)
+    (property "Datasheet" "~" (at 230.505 52.705 0)
       (effects (font (size 1.27 1.27)) hide)
     )
@@
       (effects (font (size 1.27 1.27)))
     )
-    (property "Footprint" "bitaxe:TPS40305" (at 108.585 54.61 0)
+    (property "Footprint" "TPS40305_supply:TPS40305" (at 108.585 54.61 0)
       (effects (font (size 1.27 1.27)) hide)
     )
@@
       (effects (font (size 1.27 1.27)) (justify left))
     )
-    (property "Footprint" "bitaxe:CSD17311Q5" (at 185.42 53.34 0)
+    (property "Footprint" "TPS40305_supply:CSD17311Q5" (at 185.42 53.34 0)
       (effects (font (size 1.27 1.27)) hide)
     )
@@
       (effects (font (size 1.27 1.27)) hide)
     )
-    (property "Datasheet" "" (at 145.415 37.465 0)
+    (property "Datasheet" "~" (at 145.415 37.465 0)
       (effects (font (size 1.27 1.27)) hide)
     )
@@
       (effects (font (size 1.27 1.27)) (justify left))
     )
-    (property "Footprint" "Package_TO_SOT_SMD:SOT-323_SC-70" (at 73.66 63.373 0)
+    (property "Footprint" "Package_TO_SOT_SMD:SOT-23" (at 73.66 63.373 0)
       (effects (font (size 1.27 1.27) italic) (justify left) hide)
     )
@@
       (effects (font (size 1.27 1.27)) hide)
     )
-    (property "Datasheet" "" (at 193.04 118.11 0)
+    (property "Datasheet" "~" (at 193.04 118.11 0)
       (effects (font (size 1.27 1.27)) hide)
     )
@@
       (effects (font (size 1.27 1.27)) (justify left))
     )
-    (property "Footprint" "bitaxe:CSD17311Q5" (at 185.42 27.94 0)
+    (property "Footprint" "TPS40305_supply:CSD17311Q5" (at 185.42 27.94 0)
       (effects (font (size 1.27 1.27)) hide)
     )
@@
       (effects (font (size 1.27 1.27)) hide)
     )
-    (property "Datasheet" "https://www.eaton.com/content/dam/eaton/products/electronic-components/resources/data-sheet/eaton-fp1005r-high-current-power-inductors-data-sheet.pdf" (at 189.23 39.37 0)
+    (property "Datasheet" "~" (at 189.23 39.37 0)
       (effects (font (size 1.27 1.27)) hide)
     )
@@
       (effects (font (size 1.27 1.27)) hide)
     )
-    (property "Datasheet" "" (at 45.085 136.525 0)
-      (effects (font (size 1.27 1.27)) hide)
-    )
+    (property "Datasheet" "~" (at 45.085 136.525 0)
+      (effects (font (size 1.27 1.27)) hide)
+    )
